File: Iteration_2/Project_Files/digital_voltmeter-2025-10-26_101858/digital_voltmeter.kicad_sch (KiCad schematic)
At the start: 31 parts, among them J1 Screw_Terminal_01x02, J2 Screw_Terminal_01x02, J3 ICL_7107_Conn_02x20_Counter_C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, J4 LM555_Conn_02x04_Counter_Cloc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, U3 LM7805_TO220, U4 SA39-11EWA, U5 SA39-11EWA, U6 SA39-11EWA, U7 SA39-11EWA

Commit message: commit
Connections:
- net GND: now also J2.1 (Pin_1)
- net VCC: now also J2.2 (Pin_2)
- net at J1.1 (Pin_1), R10.2: no longer J2.1 (Pin_1)
- net at C7.2, J1.2 (Pin_2), J3.30 (Pin_30)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: no longer J2.2 (Pin_2)
Other:
- moved on the sheet: J2
Changed lines of the file:
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@@
 	)
 	(junction
-		(at 196.85 91.44)
+		(at 189.23 50.8)
 		(diameter 0)
 		(color 0 0 0 0)
@@
 	)
 	(junction
+		(at 207.01 60.96)
+		(diameter 0)
+		(color 0 0 0 0)
+	)
+	(junction
 		(at 167.64 111.76)
 		(diameter 0)
@@
 	)
 	(junction
-		(at 196.85 111.76)
-		(diameter 0)
-		(color 0 0 0 0)
-	)
-	(junction
 		(at 144.78 135.89)
 		(diameter 0)
@@
 	(wire
 		(pts
+			(xy 189.23 50.8) (xy 195.58 50.8)
+		)
+		(stroke
+			(width 0)
+			(type default)
+		)
+	)
+	(wire
+		(pts
 			(xy 90.17 147.32) (xy 105.41 147.32)
 		)
@@
 	(wire
 		(pts
-			(xy 189.23 50.8) (xy 195.58 50.8)
-		)
-		(stroke
-			(width 0)
-			(type default)
-		)
-	)
-	(wire
-		(pts
 			(xy 53.34 121.92) (xy 64.77 121.92)
 		)
@@
 	(wire
 		(pts
-			(xy 229.87 91.44) (xy 196.85 91.44)
-		)
-		(stroke
-			(width 0)
-			(type default)
-		)
-	)
-	(wire
-		(pts
 			(xy 106.68 157.48) (xy 128.27 157.48)
 		)
@@
 	(wire
 		(pts
-			(xy 229.87 102.87) (xy 229.87 111.76)
-		)
-		(stroke
-			(width 0)
-			(type default)
-		)
-	)
-	(wire
-		(pts
 			(xy 220.98 50.8) (xy 220.98 40.64)
 		)
@@
 	(wire
 		(pts
-			(xy 229.87 111.76) (xy 196.85 111.76)
-		)
-		(stroke
-			(width 0)
-			(type default)
-		)
-	)
-	(wire
-		(pts
 			(xy 167.64 91.44) (xy 154.94 91.44)
 		)
@@
 	(wire
 		(pts
+			(xy 176.53 50.8) (xy 189.23 50.8)
+		)
+		(stroke
+			(width 0)
+			(type default)
+		)
+	)
+	(wire
+		(pts
 			(xy 53.34 167.64) (xy 64.77 167.64)
 		)
@@
 	(wire
 		(pts
-			(xy 229.87 100.33) (xy 229.87 91.44)
-		)
-		(stroke
-			(width 0)
-			(type default)
-		)
-	)
-	(wire
-		(pts
 			(xy 144.78 111.76) (xy 144.78 135.89)
 		)
@@
 	(wire
 		(pts
-			(xy 207.01 58.42) (xy 207.01 64.77)
+			(xy 207.01 58.42) (xy 207.01 60.96)
 		)
 		(stroke
@@
 	(wire
 		(pts
+			(xy 176.53 60.96) (xy 207.01 60.96)
+		)
+		(stroke
+			(width 0)
+			(type default)
+		)
+	)
+	(wire
+		(pts
 			(xy 154.94 86.36) (xy 154.94 91.44)
 		)
@@
 	(wire
 		(pts
+			(xy 207.01 60.96) (xy 207.01 64.77)
+		)
+		(stroke
+			(width 0)
+			(type default)
+		)
+	)
+	(wire
+		(pts
 			(xy 104.14 30.48) (xy 104.14 33.02)
 		)
@@
 		(pts
 			(xy 53.34 142.24) (xy 64.77 142.24)
+		)
+		(stroke
+			(width 0)
+			(type default)
+		)
+	)
+	(wire
+		(pts
+			(xy 176.53 53.34) (xy 176.53 60.96)
 		)
 		(stroke
@@
 	(symbol
 		(lib_id "Connector:Screw_Terminal_01x02")
-		(at 234.95 100.33 0)
+		(at 171.45 53.34 180)
 		(unit 1)
 		(exclude_from_sim no)
@@
 		(fields_autoplaced yes)
 		(property "Reference" "J2"
-			(at 237.49 100.3299 0)
-			(effects
-				(font
-					(size 1.27 1.27)
-				)
-				(justify left)
+			(at 171.45 44.45 0)
+			(effects
+				(font
+					(size 1.27 1.27)
+				)
 			)
 		)
 		(property "Value" "Screw_Terminal_01x02"
-			(at 237.49 102.8699 0)
-			(effects
-				(font
-					(size 1.27 1.27)
-				)
-				(justify left)
+			(at 171.45 46.99 0)
+			(effects
+				(font
+					(size 1.27 1.27)
+				)
 			)
 		)
 		(property "Footprint" "TerminalBlock_Phoenix:TerminalBlock_Phoenix_MKDS-1,5-2_1x02_P5.00mm_Horizontal"
-			(at 234.95 100.33 0)
+			(at 171.45 53.34 0)
 			(effects
 				(font
@@
 		)
 		(property "Datasheet" "~"
-			(at 234.95 100.33 0)
+			(at 171.45 53.34 0)
 			(effects
 				(font
@@
 		)
 		(property "Description" "Generic screw terminal, single row, 01x02, script generated (kicad-library-utils/schlib/autogen/connector/)"
-			(at 234.95 100.33 0)
+			(at 171.45 53.34 0)
 			(effects
 				(font
@@
 		)
 		(instances
-			(project ""
+			(project "digital_voltmeter"
 				(path "/32a50b93-bc82-4a95-a6b7-0296890258fa"
 					(reference "J2")
